File: hw/ferrit-m8/sxa.kicad_sch (KiCad schematic)
At the start: 30 parts, among them J1 Conn_02x10_Odd_Even, U1 74LS138

Commit message: cleanup schematics
Other:
- note added: "FERRIT-M"
- note removed: "FERRIT-K"
- company: (none) -> Copyright © 2026 Lone Dynamics Corporation
- title: (none) -> Ferrit Backplane
Changed lines of the file:
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@@
 	(generator_version "8.0")
 	(paper "A2")
+	(title_block
+		(title "Ferrit Backplane")
+		(date "2026-03-18")
+		(company "Copyright © 2026 Lone Dynamics Corporation")
+	)
 	(junction
 		(at 184.15 39.37)
@@
 		)
 	)
-	(text "FERRIT-K"
+	(text "FERRIT-M"
 		(exclude_from_sim no)
 		(at 476.25 387.35 0)

Commit message: cleanup schematics
Other:
- title: Ferrit Backplane -> Ferrit Memory Card (8 x SOP-16)
Changed lines of the file:
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@@
 	(paper "A2")
 	(title_block
-		(title "Ferrit Backplane")
+		(title "Ferrit Memory Card (8 x SOP-16)")
 		(date "2026-03-18")
 		(company "Copyright © 2026 Lone Dynamics Corporation")
