File: hw/ferrit-16/ssu.kicad_pcb (KiCad board)
At the start: 4 copper layers, 90 x 90 mm, 40 parts, among them J1 Conn_02x10_Odd_Even, J10 Conn_02x10_Odd_Even, J11 Conn_02x10_Odd_Even, J12 Conn_02x10_Odd_Even, J13 Conn_02x10_Odd_Even, J14 Conn_02x10_Odd_Even, J15 Conn_02x10_Odd_Even, J16 Conn_02x10_Odd_Even, J17 Conn_02x10_Odd_Even, J2 Conn_02x10_Odd_Even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

Commit message: update designs
Parts:
- removed SW1: BOOT, LD-SWITCH:Kailh_Mute_6x6mm
- added G***: LOGO, LD-LOGO:ld-kicad, B.Cu at (145.1, 86.7)
Connections:
- J17 pad 2: /SS0 -> /SS
- J17 pad 4: /BOOT -> /SS0
- U1 pad 19: GND -> /SS
Routing:
- net /SS: track 0.00 -> 54.5 mm
- net /BOOT: track 28.7 -> 0.00 mm
- net /SS0: track 45.1 -> 42.8 mm
- net GND: track 42.1 -> 40.8 mm
- net /KQSPI_SS12: track 54.7 -> 54.0 mm
Other:
- board text added: "V0"
