File: hw/ferrit-16/ssu.kicad_sch (KiCad schematic)
At the start: 40 parts, among them J1 Conn_02x10_Odd_Even, J10 Conn_02x10_Odd_Even, J11 Conn_02x10_Odd_Even, J12 Conn_02x10_Odd_Even, J13 Conn_02x10_Odd_Even, J14 Conn_02x10_Odd_Even, J15 Conn_02x10_Odd_Even, J16 Conn_02x10_Odd_Even, J17 Conn_02x10_Odd_Even, J2 Conn_02x10_Odd_Even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

Commit message: cleanup schematics
Other:
- company: (none) -> Copyright © 2026 Lone Dynamics Corporation
- title: (none) -> Ferrit -M8 Memory Card (8 x SOP-16)
Changed lines of the file:
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@@
 	(generator_version "8.0")
 	(paper "A1")
+	(title_block
+		(title "Ferrit -M8 Memory Card (8 x SOP-16)")
+		(date "2026-03-07")
+		(rev "V0")
+		(company "Copyright © 2026 Lone Dynamics Corporation")
+	)
 	(wire
 		(pts
@@
 	(text "FERRIT-16\nU B E R S T A H L"
 		(exclude_from_sim no)
-		(at 722.63 563.372 0)
+		(at 722.63 561.34 0)
 		(effects
 			(font
-				(size 3.81 3.81)
+				(size 3.175 3.175)
 				(thickness 1)
 				(bold yes)

Commit message: cleanup schematics
Other:
- note added: "FERRIT-16"
- note added: "U B E R S T A H L"
- note removed: "FERRIT-16 U B E R S T A H L"
- title: Ferrit -M8 Memory Card (8 x SOP-16) -> Ferrit Backplane
Changed lines of the file:
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@@
 	(paper "A1")
 	(title_block
-		(title "Ferrit -M8 Memory Card (8 x SOP-16)")
+		(title "Ferrit Backplane")
 		(date "2026-03-07")
 		(rev "V0")
@@
 		)
 	)
-	(text "FERRIT-16\nU B E R S T A H L"
+	(text "U B E R S T A H L"
 		(exclude_from_sim no)
 		(at 722.63 561.34 0)
 		(effects
 			(font
-				(size 3.175 3.175)
+				(size 1.905 1.905)
+				(thickness 1)
+				(bold yes)
+			)
+			(justify left bottom)
+		)
+	)
+	(text "FERRIT-16"
+		(exclude_from_sim no)
+		(at 721.868 557.276 0)
+		(effects
+			(font
+				(size 3.81 3.81)
 				(thickness 1)
 				(bold yes)

Commit message: update designs
Parts:
- removed SW3: BOOT, LD-SWITCH:Kailh_Mute_6x6mm, symbol Switch:SW_Push
Connections:
- net BOOT is gone; now on net SS0: J17.4 (Pin_4)
- net GND: no longer U1.19 (E1)
- net SS0: no longer J17.2 (Pin_2)
- new net SS: J17.2 (Pin_2), U1.19 (E1)
Changed lines of the file:
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@@
 	(wire
 		(pts
-			(xy 764.54 99.06) (xy 773.43 99.06)
-		)
-		(stroke
-			(width 0)
-			(type default)
-		)
-	)
-	(wire
-		(pts
 			(xy 83.82 275.59) (xy 100.33 275.59)
 		)
@@
 	(wire
 		(pts
-			(xy 789.94 99.06) (xy 783.59 99.06)
-		)
-		(stroke
-			(width 0)
-			(type default)
-		)
-	)
-	(wire
-		(pts
 			(xy 139.7 143.51) (xy 156.21 143.51)
 		)
@@
 	(wire
 		(pts
-			(xy 764.54 93.98) (xy 764.54 99.06)
-		)
-		(stroke
-			(width 0)
-			(type default)
-		)
-	)
-	(wire
-		(pts
 			(xy 139.7 138.43) (xy 156.21 138.43)
 		)
@@
 	)
 	(label "SS0"
-		(at 99.06 74.93 180)
+		(at 99.06 77.47 180)
 		(effects
 			(font
@@
 		)
 	)
-	(label "BOOT"
-		(at 767.08 99.06 0)
-		(effects
-			(font
-				(size 1.27 1.27)
-			)
-			(justify left bottom)
-		)
-	)
 	(label "KQSPI_SS9"
 		(at 241.3 297.18 180)
@@
 		)
 	)
-	(label "BOOT"
-		(at 99.06 77.47 180)
+	(label "SS"
+		(at 99.06 74.93 180)
 		(effects
 			(font
@@
 		)
 	)
-	(label "GND"
+	(label "SS"
 		(at 182.88 289.56 0)
 		(effects
@@
 		)
 	)
-	(symbol
-		(lib_id "Switch:SW_Push")
-		(at 778.51 99.06 0)
-		(unit 1)
-		(exclude_from_sim no)
-		(in_bom yes)
-		(on_board yes)
-		(dnp no)
-		(property "Reference" "SW3"
-			(at 778.51 91.821 0)
-			(effects
-				(font
-					(size 1.27 1.27)
-				)
-			)
-		)
-		(property "Value" "BOOT"
-			(at 778.51 94.1324 0)
-			(effects
-				(font
-					(size 1.27 1.27)
-				)
-			)
-		)
-		(property "Footprint" "LD-SWITCH:Kailh_Mute_6x6mm"
-			(at 778.51 93.98 0)
-			(effects
-				(font
-					(size 1.27 1.27)
-				)
-				(hide yes)
-			)
-		)
-		(property "Datasheet" "~"
-			(at 778.51 93.98 0)
-			(effects
-				(font
-					(size 1.27 1.27)
-				)
-				(hide yes)
-			)
-		)
-		(property "Description" ""
-			(at 778.51 99.06 0)
-			(effects
-				(font
-					(size 1.27 1.27)
-				)
-				(hide yes)
-			)
-		)
-		(pin "1"
-		)
-		(pin "2"
-		)
-		(instances
-			(project ""
-				(path "/3c9169cc-3a77-4ae0-8afc-cbfc472a28c5"
-					(reference "SW3")
-					(unit 1)
-				)
-			)
-			(project "ssu"
-				(path "/86ed1906-88c0-4113-ab7c-ce662689fe6d"
-					(reference "SW1")
-					(unit 1)
-				)
-			)
-			(project "ldp"
-				(path "/aeaf2554-c305-426e-a20b-1d2ccb0e55e2"
-					(reference "SW3")
-					(unit 1)
-				)
-			)
-		)
-	)
-	(symbol
-		(lib_id "power:GND")
-		(at 789.94 99.06 0)
-		(unit 1)
-		(exclude_from_sim no)
-		(in_bom yes)
-		(on_board yes)
-		(dnp no)
-		(property "Reference" "#PWR033"
-			(at 789.94 105.41 0)
-			(effects
-				(font
-					(size 1.27 1.27)
-				)
-				(hide yes)
-			)
-		)
-		(property "Value" "GND"
-			(at 790.067 103.4542 0)
-			(effects
-				(font
-					(size 1.27 1.27)
-				)
-			)
-		)
-		(property "Footprint" ""
-			(at 789.94 99.06 0)
-			(effects
-				(font
-					(size 1.27 1.27)
-				)
-				(hide yes)
-			)
-		)
-		(property "Datasheet" ""
-			(at 789.94 99.06 0)
-			(effects
-				(font
-					(size 1.27 1.27)
-				)
-				(hide yes)
-			)
-		)
-		(property "Description" ""
-			(at 789.94 99.06 0)
-			(effects
-				(font
-					(size 1.27 1.27)
-				)
-				(hide yes)
-			)
-		)
-		(pin "1"
-		)
-		(instances
-			(project ""
-				(path "/3c9169cc-3a77-4ae0-8afc-cbfc472a28c5"
-					(reference "#PWR033")
-					(unit 1)
-				)
-			)
-			(project "ssu"
-				(path "/86ed1906-88c0-4113-ab7c-ce662689fe6d"
-					(reference "#PWR26")
-					(unit 1)
-				)
-			)
-			(project "ldp"
-				(path "/aeaf2554-c305-426e-a20b-1d2ccb0e55e2"
-					(reference "#PWR033")
-					(unit 1)
-				)
-			)
-		)
-	)
