File: hw/ferrit-cy/sxy.kicad_pcb (KiCad board)
At the start: 4 copper layers, 27.8 x 44 mm, 45 parts, among them J1 USB_C_Receptacle_USB2.0_16P, J3 Conn_02x10_Odd_Even, U1 RP2040, U2 TLV62568DDC, U3 W25Q32JVSS, Y2 ECS-80-12-33-JGN-TR-12MHZ

Commit message: update designs
Parts:
- added SW3: BOOT, LD-SWITCH:Button_2P_3x4mm, F.Cu at (113.9, 94.5)
- R10, R9: footprint Resistor_SMD:R_0603_1608Metric -> Resistor_SMD:R_0402_1005Metric
- R11: value 210K -> 200K
- R12: value 47K -> 44K2
- U3: value W25Q32JVSS -> M95P32-IXMNT/E
- moved R10 2.58 mm to (118.0, 93.6)
- moved R9 2.58 mm to (118.0, 95.2)
Connections:
- J3 pad 2: /SS0 -> /SS
- J3 pad 4: /BOOT -> /KSS0
- RN1 pad 4: unconnected-(RN1-R4.1-Pad4) -> /SS0
- RN1 pad 5: unconnected-(RN1-R4.2-Pad5) -> /KSS0
- U1 pad 3: unconnected-(U1-GPIO1-Pad3) -> /SS
Routing:
- net /BOOT: track 9.45 -> 40.3 mm
- net /SS: track 0.00 -> 19.0 mm
- net /SS0: track 19.1 -> 3.16 mm
- net /KSS0: track 0.00 -> 14.1 mm
- net /USBC_CC2: track 10.6 -> 6.56 mm
- net /USBC_CC1: track 12.1 -> 8.80 mm
- net GND: track 31.0 -> 31.9 mm, vias 35 -> 36
- net /USBCDP: track 23.5 -> 22.9 mm
- net /USBCDN: track 21.8 -> 21.2 mm

Commit message: update designs
Parts:
- SW3: footprint LD-SWITCH:Button_2P_3x4mm -> LD-SWITCH:SW_SMD_2P_3X6MM
- moved R10 16.2 mm to (121.6, 109.4)
- moved R9 15.7 mm to (121.6, 110.4)
- moved F1 0.60 mm to (115.3, 97.9)
- moved FB1 0.60 mm to (115.3, 99.7)
- moved SW3 0.23 mm to (113.9, 94.2)
Routing:
- net /USBC_CC2: track 6.56 -> 12.3 mm
- net GND: track 31.9 -> 29.2 mm, vias 36 -> 34
- net /USBC_CC1: track 8.80 -> 10.7 mm
- net /BOOT: track 40.3 -> 39.4 mm
