File: hw/ferrit-cy/sxy.kicad_sch (KiCad schematic)
At the start: 45 parts, among them J1 USB_C_Receptacle_USB2.0_16P, J3 Conn_02x10_Odd_Even, U1 RP2040, U2 TLV62568DDC, U3 W25Q32JVSS, Y2 ECS-80-12-33-JGN-TR-12MHZ

Commit message: cleanup schematics
Parts:
- R11: value 210K -> 200K
- R12: value 47K -> 44K2
- U3: value W25Q32JVSS -> M95P32-IXMNT/E
Other:
- note added: "0.6 * (1 + (200/44.2)) = 3.3149"
- note removed: "0.6 * (1 + (210/47)) = 3.28"
- company: (none) -> Copyright © 2026 Lone Dynamics Corporation
- title: (none) -> Ferrit Controller Model Y
Changed lines of the file:
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@@
 	(generator_version "8.0")
 	(paper "A1")
+	(title_block
+		(title "Ferrit Controller Model Y")
+		(date "2026-03-19")
+		(rev "V0")
+		(company "Copyright © 2026 Lone Dynamics Corporation")
+	)
 	(junction
 		(at 73.66 58.42)
@@
 	(wire
 		(pts
-			(xy 160.02 121.92) (xy 161.29 121.92)
-		)
-		(stroke
-			(width 0)
-			(type default)
-		)
-	)
-	(wire
-		(pts
 			(xy 134.62 176.53) (xy 118.11 176.53)
 		)
@@
 		)
 	)
-	(text "0.6 * (1 + (210/47)) = 3.28"
+	(text "0.6 * (1 + (200/44.2)) = 3.3149"
 		(exclude_from_sim no)
 		(at 687.07 495.3 0)
@@
 	)
 	(label "PWR3V3"
-		(at 161.29 128.27 90)
+		(at 161.29 121.92 270)
 		(effects
 			(font
 				(size 1.27 1.27)
 			)
-			(justify left bottom)
+			(justify right bottom)
 		)
 	)
@@
 			)
 		)
-		(property "Value" "210K"
+		(property "Value" "200K"
 			(at 678.688 510.413 0)
 			(effects
@@
 			)
 		)
-		(property "Value" "47K"
+		(property "Value" "44K2"
 			(at 678.688 534.543 0)
 			(effects
@@
 		(fields_autoplaced yes)
 		(property "Reference" "U3"
-			(at 221.7294 117.094 0)
+			(at 221.9041 116.84 0)
 			(effects
 				(font
@@
 			)
 		)
-		(property "Value" "W25Q32JVSS"
-			(at 221.7294 119.634 0)
+		(property "Value" "M95P32-IXMNT/E"
+			(at 221.9041 119.38 0)
 			(effects
 				(font

Commit message: update designs
Parts:
- added SW3: BOOT, LD-SWITCH:Button_2P_3x4mm, symbol Switch:SW_Push
- R10, R9: footprint Resistor_SMD:R_0603_1608Metric -> Resistor_SMD:R_0402_1005Metric
Connections:
- net BOOT: now also SW3.1; no longer J3.4 (Pin_4)
- net GND: now also SW3.2
- net SS0: now also RN1.4 (R4.1); no longer J3.2 (Pin_2)
- net KSS0: now reaches RN1.5 (R4.2)
- net KSS0: now also J3.4 (Pin_4)
- net SS: now reaches U1.3 (GPIO1)
- net SS: now also J3.2 (Pin_2)
Other:
- moved on the sheet: C1, C10, C11, C12, C13, C14, C15, C16, C17, C18, C19, C2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

Commit message: update designs
Parts:
- SW3: footprint LD-SWITCH:Button_2P_3x4mm -> LD-SWITCH:SW_SMD_2P_3X6MM
Changed lines of the file:
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@@
 			)
 		)
-		(property "Footprint" "LD-SWITCH:Button_2P_3x4mm"
+		(property "Footprint" "LD-SWITCH:SW_SMD_2P_3X6MM"
 			(at 594.614 108.712 0)
 			(effects
